File: MainBoard PB/MainBoardPB/MainBoardPB.kicad_pcb (KiCad board)
At the start: 2 copper layers, 202.3 x 50.1 mm, 39 parts, among them J1 Conn_01x02, J3 Conn_01x02, J7 Conn_01x04, J8 Conn_01x02, Q6 BC817, Q7 BC817, U6 PC817, U7 PC817

Commit message: ADD ALL PLEASE DURA EBANAYA
Parts:
- removed the G*** at (189.0, 73.2)
- removed the J1 at (195.6, 91.2)
- removed the J3 at (262.5, 86.3)
- removed the J7 at (262.9, 105.2)
- removed the J8 at (242.9, 108.0)
- removed the Q6 at (240.7, 82.5)
- removed the Q7 at (240.6, 97.3)
- removed the R10 at (240.6, 93.8)
- removed the R11 at (242.5, 87.0)
- removed the R12 at (239.7, 101.6)
- removed the R7 at (254.9, 87.7)
- removed the R8 at (254.0, 101.7)
- removed the R9 at (241.1, 79.6)
- removed the U6 at (250.1, 82.8)
- removed the U7 at (249.2, 97.5)
- removed the VD1 at (203.3, 91.3)
- removed the VD2 at (218.5, 97.4)
- removed the VS1 at (234.8, 82.2)
- removed the VS2 at (223.8, 97.6)
- moved J7 71.6 mm to (109.0, 54.7)
- moved R10 71.6 mm to (86.7, 43.3)
- moved R7 71.6 mm to (101.0, 37.2)
- moved R8 71.6 mm to (100.1, 51.2)
- moved R9 71.6 mm to (87.2, 29.1)
- moved VD2 71.6 mm to (64.7, 46.9)
- moved G*** 71.6 mm to (35.2, 22.6)
- moved J1 71.6 mm to (41.8, 40.8)
- moved J3 71.6 mm to (108.6, 35.8)
- moved J8 71.6 mm to (89.0, 57.5)
- moved Q6 71.6 mm to (86.9, 32.0)
- moved Q7 71.6 mm to (86.7, 46.8)
- moved R11 71.6 mm to (88.7, 36.5)
- moved R12 71.6 mm to (85.8, 51.1)
- moved U6 71.6 mm to (96.2, 32.3)
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Routing:
- net /DC_+: track 241.1 -> 120.6 mm
- net /L: track 180.1 -> 90.0 mm
- net /DC_-: track 125.3 -> 62.6 mm
- net GND: track 83.2 -> 41.6 mm
- net +5V: track 72.8 -> 36.4 mm
- net /Tyr1REG: track 67.4 -> 33.7 mm, vias 4 -> 2
- net /Tyr_G1: track 50.8 -> 25.4 mm
- net /N: track 27.7 -> 13.9 mm
- net /Tyr2REG: track 27.0 -> 13.5 mm
- net GND1: track 26.7 -> 13.3 mm, vias 4 -> 2
- net Net-(Q6-B): track 24.7 -> 12.4 mm
- net Net-(Q7-B): track 22.8 -> 11.4 mm
- net /Tyr_G2: track 16.5 -> 8.27 mm
- net Net-(R7-Pad1): track 7.33 -> 3.66 mm
- net Net-(R8-Pad1): track 5.74 -> 2.87 mm
Other:
- board size 202.3 x 50.1 mm -> 99.1 x 50 mm
