File: MainBoard PB/MainBoardPB/MainBoardPB.kicad_sch (KiCad schematic)
At the start: 64 parts, among them J1 Conn_01x02, J2 Conn_01x03, J3 Conn_01x02, J4 Conn_01x02, J5 Conn_01x02, J6 Conn_01x03, J7 Conn_01x04, J8 Conn_01x02, Q6 BC817, Q7 BC817, SW4 KLS7-TS3401, T1 Transformer_1P_1S, U1 IRM-02-5, U6 PC817, U7 PC817, Y1 25 MHz, Y2 32.7 kHz

Commit message: ADD ALL PLEASE DURA EBANAYA
Parts:
- added DD2: RFM98W-433S2, RF_Module:HOPERF_RFM9XW_SMD, symbol RF_Module:RFM98W-433S2
- added DD3_TFT: CR2013-MI2120, Display:CR2013-MI2120, symbol Driver_Display:CR2013-MI2120
- DD2: value ESP-07 -> RFM98W-433S2; footprint RF_Module:ESP-07 -> RF_Module:HOPERF_RFM9XW_SMD
- renumbered C23 to C23_32CLK, C24 to C24_32CLK, C4 to C4_OUTFLTR, C5 to C5_OUTFLTR, C6 to C6_CLK, C7 to C7_CLK, L1 to L1_OUTFLTR
Connections:
- net SPI_SCK: now reaches DD1.29 (PA5)
- net SPI_MISO: now reaches DD1.30 (PA6)
- net SPI_MOSI: now reaches DD1.31 (PA7)
- net UART_RX: now reaches DD1.70 (PA11)
- net UART_TX: now reaches DD1.71 (PA12)
- net SWO: now reaches DD1.89 (PB3(JTDO)
Changed lines of the file:
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@@
 	(generator "eeschema")
 	(generator_version "10.0")
-	(paper "A3")
+	(paper "A2")
